Commit message: them muc thiu

File: urdf/stl.urdf (robot description, URDF)
Before this commit: robot robot_name, 5 links, 4 joints
Links:
- removed link base_link_2
- removed link base_link_3
- removed link base_link_4
- removed link base_link_5
- added link Lidar_link, mass 97.167; collision mesh filename=package://Assem1/meshes/Lidar_link.STL; visual mesh filename=package://Assem1/meshes/Lidar_link.STL
- added link banh1_Link, mass 12.33; collision mesh filename=package://Assem1/meshes/banh1_Link.STL; visual mesh filename=package://Assem1/meshes/banh1_Link.STL
- added link banh2_Link, mass 12.33; collision mesh filename=package://Assem1/meshes/banh2_Link.STL; visual mesh filename=package://Assem1/meshes/banh2_Link.STL
- added link banh3_Link, mass 12.33; collision mesh filename=package://Assem1/meshes/banh3_Link.STL; visual mesh filename=package://Assem1/meshes/banh3_Link.STL
- added link banh4_Link, mass 12.33; collision mesh filename=package://Assem1/meshes/banh4_Link.STL; visual mesh filename=package://Assem1/meshes/banh4_Link.STL
- link base_link: mass None -> 1600.6; geometry collision mesh filename=package://Assem1/meshes/base_link.STL; visual mesh filename=package://Assem1/meshes/base_link.STL
Joints:
- removed joint base_link_to_base_link_2
- removed joint base_link_to_base_link_3
- removed joint base_link_to_base_link_4
- removed joint base_link_to_base_link_5
- added joint LiDar joint: type fixed, parent base_link, child Lidar_link, origin xyz=0.7375 0 0 rpy=0 0 0, axis 0 0 0
- added joint banh1 joint: type continuous, parent base_link, child banh1_Link, origin xyz=0.7375 0 0 rpy=0 0 0, axis 0 0 -1, limit effort=10 velocity=5
- added joint banh2 joint: type continuous, parent base_link, child banh2_Link, origin xyz=0.7375 0 0 rpy=0 0 0, axis 0 0 1, limit effort=10 velocity=5
- added joint banh3 joint: type continuous, parent base_link, child banh3_Link, origin xyz=0.7375 0 0 rpy=0 0 0, axis 0 0 1, limit effort=10 velocity=5
- added joint banh4 joint: type continuous, parent base_link, child banh4_Link, origin xyz=0.7375 0 0 rpy=0 0 0, axis 0 0 -1, limit effort=10 velocity=5
